File: V1/RJ45-breakout_1ch-V1.kicad_pcb (KiCad board)
At the start: 2 copper layers, 22.9 x 30.5 mm, 2 parts, among them J1 RJ45, J2 Screw_Terminal_01x04

Commit message: kicad version conversion
Other:
- net class Default removed
