File: V1/RJ45-breakout_1ch-V1.kicad_pcb (KiCad board)
At the start: 2 copper layers, 22.9 x 30.5 mm, 2 parts, among them J1 RJ45, J2 Screw_Terminal_01x04

Commit message: work in progress
Parts:
- moved J1 74.5 mm to (144.8, 92.7)
- moved J2 74.5 mm to (141.0, 108.0)
Other:
- board text added: "+V"
- board text added: "1x RJ45 BRKOUT"
- board text added: "SW1"
- board text added: "SW2"
- board text added: "SW3"
- board text removed: "1x RJ45 BREAKOUT"
Changed lines of the file:
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@@
   (setup
     (pad_to_mask_clearance 0)
-    (aux_axis_origin 64.77 132.08)
+    (aux_axis_origin 137.16 114.3)
     (pcbplotparams
       (layerselection 0x00010e0_ffffffff)
@@
   (net 4 "Net-(J1-Pad7)")
   (footprint "Tales:RJ45_Amphenol_RJHSE5080" (layer "F.Cu")
-    (at 72.39 110.49)
+    (at 144.78 92.71)
     (descr "Unshielded")
     (tags "RJ45 8p8c ethernet cat5")
@@
       (effects (font (size 1 1) (thickness 0.15)))
     )
-    (fp_text value "RJ45" (at 3.56 9.5) (layer "F.Fab")
+    (fp_text value "RJ45" (at 3.56 -3.81) (layer "F.Fab")
       (effects (font (size 1 1) (thickness 0.15)))
     )
@@
   )
   (footprint "Tales:TerminalBlock_Phoenix_MKDS-3-4-5.08_1x04_P5.08mm_Horizontal" (layer "F.Cu")
-    (at 68.58 125.73)
+    (at 140.97 107.95)
     (descr "Terminal Block Phoenix MKDS-3-4-5.08, 4 pins, pitch 5.08mm, size 20.3x11.2mm^2, drill diamater 1.3mm, pad diameter 2.6mm, see http://www.farnell.com/datasheets/2138224.pdf, script-generated using https://github.com/pointhi/kicad-footprint-generator/scripts/TerminalBlock_Phoenix")
     (tags "THT Terminal Block Phoenix MKDS-3-4-5.08 pitch 5.08mm size 20.3x11.2mm^2 drill 1.3mm pad 2.6mm")
@@
       (effects (font (size 1 1) (thickness 0.15)))
     )
-    (fp_text value "Screw_Terminal_01x04" (at 7.62 6.36) (layer "F.Fab")
-      (effects (font (size 1 1) (thickness 0.15)))
-    )
-    (fp_text user "${REFERENCE}" (at 7.62 3.1) (layer "F.Fab")
+    (fp_text value "Screw_Terminal_01x04" (at 7.62 -3.175) (layer "F.Fab")
+      (effects (font (size 1 1) (thickness 0.15)))
+    )
+    (fp_text user "${REFERENCE}" (at 7.62 -5.08) (layer "F.Fab")
       (effects (font (size 1 1) (thickness 0.15)))
     )
@@
     )
   )
-  (gr_line (start 64.77 132.08) (end 87.63 132.08) (layer "Edge.Cuts") (width 0.1))
-  (gr_line (start 64.77 101.6) (end 64.77 132.08) (layer "Edge.Cuts") (width 0.1))
-  (gr_line (start 87.63 101.6) (end 64.77 101.6) (layer "Edge.Cuts") (width 0.1))
-  (gr_line (start 87.63 132.08) (end 87.63 101.6) (layer "Edge.Cuts") (width 0.1))
-  (gr_text "1x RJ45 BREAKOUT" (at 66.675 109.855 90) (layer "F.SilkS")
+  (gr_line (start 137.16 114.3) (end 160.02 114.3) (layer "Edge.Cuts") (width 0.1))
+  (gr_line (start 137.16 83.82) (end 137.16 114.3) (layer "Edge.Cuts") (width 0.1))
+  (gr_line (start 160.02 83.82) (end 137.16 83.82) (layer "Edge.Cuts") (width 0.1))
+  (gr_line (start 160.02 114.3) (end 160.02 83.82) (layer "Edge.Cuts") (width 0.1))
+  (gr_text "SW2" (at 151.13 111.76) (layer "B.Cu")
+    (effects (font (size 1.5 1.2) (thickness 0.2)) (justify mirror))
+  )
+  (gr_text "+V" (at 140.97 111.76) (layer "B.Cu")
+    (effects (font (size 1.5 1.2) (thickness 0.2)) (justify mirror))
+  )
+  (gr_text "SW3" (at 156.21 111.76) (layer "B.Cu")
+    (effects (font (size 1.5 1.2) (thickness 0.2)) (justify mirror))
+  )
+  (gr_text "SW1" (at 146.05 111.76) (layer "B.Cu")
+    (effects (font (size 1.5 1.2) (thickness 0.2)) (justify mirror))
+  )
+  (gr_text "1x RJ45 BRKOUT" (at 139.065 92.075 90) (layer "F.SilkS")
     (effects (font (size 1.2 1) (thickness 0.2)))
   )
-  (gr_text "TRAMONTINA" (at 85.725 110.49 90) (layer "F.SilkS")
+  (gr_text "TRAMONTINA" (at 158.115 92.71 90) (layer "F.SilkS")
     (effects (font (size 1.2 1) (thickness 0.2)))
   )
@@
     (style (thickness 0.15) (arrow_length 1.27) (text_position_mode 0) (extension_height 0.58642) (extension_offset 0) keep_text_aligned)
   )
-  (segment (start 72.39 113.03) (end 72.39 110.49) (width 1.524) (layer "B.Cu") (net 1))
-  (segment (start 72.646 113.03) (end 72.39 113.03) (width 1.524) (layer "B.Cu") (net 1))
-  (segment (start 73.406 112.27) (end 72.646 113.03) (width 1.524) (layer "B.Cu") (net 1))
-  (segment (start 72.39 113.03) (end 72.39 115.57) (width 1.524) (layer "B.Cu") (net 1))
-  (segment (start 72.39 115.57) (end 68.58 119.38) (width 1.524) (layer "B.Cu") (net 1))
-  (segment (start 68.58 119.38) (end 68.58 125.73) (width 1.524) (layer "B.Cu") (net 1))
-  (segment (start 77.47 114.3) (end 77.47 112.27) (width 1.524) (layer "F.Cu") (net 2))
-  (segment (start 73.66 120.65) (end 77.47 116.84) (width 1.524) (layer "F.Cu") (net 2))
-  (segment (start 80.645 114.935) (end 77.47 114.935) (width 1.524) (layer "F.Cu") (net 2))
-  (segment (start 74.422 109.093) (end 75.565 107.95) (width 1.524) (layer "F.Cu") (net 2))
-  (segment (start 73.66 125.73) (end 73.66 120.65) (width 1.524) (layer "F.Cu") (net 2))
-  (segment (start 77.47 116.84) (end 77.47 114.3) (width 1.524) (layer "F.Cu") (net 2))
-  (segment (start 75.565 107.95) (end 78.559682 107.95) (width 1.524) (layer "F.Cu") (net 2))
-  (segment (start 78.559682 107.95) (end 81.915 111.305318) (width 1.524) (layer "F.Cu") (net 2))
-  (segment (start 74.422 110.49) (end 74.422 109.093) (width 1.524) (layer "F.Cu") (net 2))
-  (segment (start 81.915 111.305318) (end 81.915 113.665) (width 1.524) (layer "F.Cu") (net 2))
-  (segment (start 81.915 113.665) (end 80.645 114.935) (width 1.524) (layer "F.Cu") (net 2))
-  (segment (start 75.438 112.27) (end 75.934001 111.773999) (width 1.016) (layer "F.Cu") (net 3))
-  (segment (start 75.934001 111.009999) (end 76.454 110.49) (width 1.016) (layer "F.Cu") (net 3))
-  (segment (start 75.934001 111.773999) (end 75.934001 111.009999) (width 1.016) (layer "F.Cu") (net 3))
-  (segment (start 75.934001 111.773999) (end 75.934001 111.009999) (width 1.016) (layer "B.Cu") (net 3))
-  (segment (start 75.438 112.27) (end 75.934001 111.773999) (width 1.016) (layer "B.Cu") (net 3))
-  (segment (start 75.934001 111.009999) (end 76.454 110.49) (width 1.016) (layer "B.Cu") (net 3))
-  (segment (start 75.438 118.618) (end 78.74 121.92) (width 1.524) (layer "B.Cu") (net 3))
-  (segment (start 75.438 112.27) (end 75.438 118.618) (width 1.524) (layer "B.Cu") (net 3))
-  (segment (start 78.74 121.92) (end 78.74 125.73) (width 1.524) (layer "B.Cu") (net 3))
-  (segment (start 79.502 112.27) (end 79.502 111.506) (width 1.524) (layer "B.Cu") (net 4))
-  (segment (start 79.502 111.506) (end 78.486 110.49) (width 1.524) (layer "B.Cu") (net 4))
-  (segment (start 83.82 116.588) (end 83.82 125.73) (width 1.524) (layer "B.Cu") (net 4))
-  (segment (start 79.502 112.27) (end 83.82 116.588) (width 1.524) (layer "B.Cu") (net 4))
+  (segment (start 144.78 95.25) (end 144.78 92.71) (width 1.524) (layer "B.Cu") (net 1))
+  (segment (start 145.036 95.25) (end 144.78 95.25) (width 1.524) (layer "B.Cu") (net 1))
+  (segment (start 145.796 94.49) (end 145.036 95.25) (width 1.524) (layer "B.Cu") (net 1))
+  (segment (start 144.78 95.25) (end 144.78 97.79) (width 1.524) (layer "B.Cu") (net 1))
+  (segment (start 144.78 97.79) (end 140.97 101.6) (width 1.524) (layer "B.Cu") (net 1))
+  (segment (start 140.97 101.6) (end 140.97 107.95) (width 1.524) (layer "B.Cu") (net 1))
+  (segment (start 149.86 96.52) (end 149.86 94.49) (width 1.524) (layer "F.Cu") (net 2))
+  (segment (start 146.05 102.87) (end 149.86 99.06) (width 1.524) (layer "F.Cu") (net 2))
+  (segment (start 153.035 97.155) (end 149.86 97.155) (width 1.524) (layer "F.Cu") (net 2))
+  (segment (start 146.812 91.313) (end 147.955 90.17) (width 1.524) (layer "F.Cu") (net 2))
+  (segment (start 146.05 107.95) (end 146.05 102.87) (width 1.524) (layer "F.Cu") (net 2))
+  (segment (start 149.86 99.06) (end 149.86 96.52) (width 1.524) (layer "F.Cu") (net 2))
+  (segment (start 147.955 90.17) (end 150.949682 90.17) (width 1.524) (layer "F.Cu") (net 2))
+  (segment (start 150.949682 90.17) (end 154.305 93.525318) (width 1.524) (layer "F.Cu") (net 2))
+  (segment (start 146.812 92.71) (end 146.812 91.313) (width 1.524) (layer "F.Cu") (net 2))
+  (segment (start 154.305 93.525318) (end 154.305 95.885) (width 1.524) (layer "F.Cu") (net 2))
+  (segment (start 154.305 95.885) (end 153.035 97.155) (width 1.524) (layer "F.Cu") (net 2))
+  (segment (start 147.828 94.49) (end 148.324001 93.993999) (width 1.016) (layer "F.Cu") (net 3))
+  (segment (start 148.324001 93.229999) (end 148.844 92.71) (width 1.016) (layer "F.Cu") (net 3))
+  (segment (start 148.324001 93.993999) (end 148.324001 93.229999) (width 1.016) (layer "F.Cu") (net 3))
+  (segment (start 148.324001 93.993999) (end 148.324001 93.229999) (width 1.016) (layer "B.Cu") (net 3))
+  (segment (start 147.828 94.49) (end 148.324001 93.993999) (width 1.016) (layer "B.Cu") (net 3))
+  (segment (start 148.324001 93.229999) (end 148.844 92.71) (width 1.016) (layer "B.Cu") (net 3))
+  (segment (start 147.828 100.838) (end 151.13 104.14) (width 1.524) (layer "B.Cu") (net 3))
+  (segment (start 147.828 94.49) (end 147.828 100.838) (width 1.524) (layer "B.Cu") (net 3))
+  (segment (start 151.13 104.14) (end 151.13 107.95) (width 1.524) (layer "B.Cu") (net 3))
+  (segment (start 151.892 94.49) (end 151.892 93.726) (width 1.524) (layer "B.Cu") (net 4))
+  (segment (start 151.892 93.726) (end 150.876 92.71) (width 1.524) (layer "B.Cu") (net 4))
+  (segment (start 156.21 98.808) (end 156.21 107.95) (width 1.524) (layer "B.Cu") (net 4))
+  (segment (start 151.892 94.49) (end 156.21 98.808) (width 1.524) (layer "B.Cu") (net 4))
 )

Commit message: PCB tweaks
Parts:
- added REF**: OSHW-Logo2_7.3x6mm_Copper, Symbol:OSHW-Logo2_7.3x6mm_Copper, B.Cu at (148.6, 88.3)
Other:
- board text added: "TMASCHIO"
- board text removed: "TRAMONTINA"
