File: V1/RJ45-breakout_1ch-V1.kicad_sch (KiCad schematic)
At the start: 2 parts, among them J1 RJ45, J2 Screw_Terminal_01x04

Commit message: PCB tweaks
Other:
- title: (none) -> 1 channel RJ45 breakout board
Changed lines of the file:
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@@
 (kicad_sch (version 20211123) (generator eeschema)
   (paper "A4")
+  (title_block
+    (title "1 channel RJ45 breakout board")
+    (date "2022-04-01")
+    (rev "V1")
+  )
   (junction (at 146.05 99.06) (diameter 0) (color 0 0 0 0)
   )
