File: V1/rj45-breakout-1ch-v1.kicad_sch (KiCad schematic)
At the start: 2 parts, among them J1 RJ45, J2 1x4P 5,08 SCREW

Commit message: Renamed nets
Connections:
- net PAIR1 renamed +24V
- net PAIR2 renamed SW1
- net PAIR3 renamed SW2
- net PAIR4 renamed SW3
Other:
- note added: "J2 PIN 1 - +24V J2 PIN 2 - SWITCH 1 J2 PIN 3 - SWITCH 2 J2 PIN 4 - SWITCH 3"
- note removed: "J2 PIN 1 - 24V J2 PIN 2 - SWITCH 1 J2 PIN 3 - SWITCH 2 J2 PIN 4 - SWITCH 3"
Changed lines of the file:
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@@
 		)
 	)
-	(text "J2 PIN 1 - 24V\nJ2 PIN 2 - SWITCH 1\nJ2 PIN 3 - SWITCH 2\nJ2 PIN 4 - SWITCH 3"
+	(text "J2 PIN 1 - +24V\nJ2 PIN 2 - SWITCH 1\nJ2 PIN 3 - SWITCH 2\nJ2 PIN 4 - SWITCH 3"
 		(exclude_from_sim no)
 		(at 187.96 128.27 0)
@@
 		)
 	)
-	(label "PAIR4"
+	(label "SW3"
 		(at 154.94 104.14 0)
 		(effects
@@
 		)
 	)
-	(label "PAIR1"
+	(label "+24V"
 		(at 154.94 96.52 0)
 		(effects
@@
 		)
 	)
-	(label "PAIR2"
+	(label "SW1"
 		(at 154.94 99.06 0)
 		(effects
@@
 		)
 	)
-	(label "PAIR3"
+	(label "SW2"
 		(at 154.94 101.6 0)
 		(effects
