File: V1/rj45-breakout-1ch-v1.kicad_pcb (KiCad board)
At the start: 2 copper layers, 22 x 28 mm, 2 parts, among them J1 RJ45, J2 1x4P 5,08 SCREW

Commit message: Adjusting before fabrication
Other:
- rule pad_to_mask_clearance: 0 -> 0.1
- board text added: "+24V"
- board text removed: "+V"

Commit message: Revising before manufacturing
Parts:
- moved J2 7.50 mm to (141.0, 114.0)
- moved J1 3.64 mm to (141.0, 101.0)
Connections:
- net Net-(J2-Pin_1) renamed /PAIR1
- net Net-(J2-Pin_2) renamed /PAIR2
- net Net-(J2-Pin_3) renamed /PAIR3
- net Net-(J2-Pin_4) renamed /PAIR4
Routing:
- net /PAIR2: track 31.4 -> 29.8 mm

Commit message: Renamed nets
Connections:
- net /PAIR1 renamed /+24V
- net /PAIR2 renamed /SW1
- net /PAIR3 renamed /SW2
- net /PAIR4 renamed /SW3
Changed lines of the file:
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@@
 	)
 	(net 0 "")
-	(net 1 "/PAIR2")
-	(net 2 "/PAIR3")
-	(net 3 "/PAIR1")
-	(net 4 "/PAIR4")
+	(net 1 "/SW1")
+	(net 2 "/SW2")
+	(net 3 "/+24V")
+	(net 4 "/SW3")
 	(footprint "Tales:TerminalBlock_Dibo_DB128L-5.08-4P_1x04_P5.08mm_Horizontal"
 		(layer "F.Cu")
@@
 			(remove_unused_layers no)
 			(roundrect_rratio 0.25)
-			(net 3 "/PAIR1")
+			(net 3 "/+24V")
 			(pinfunction "Pin_1")
 			(pintype "passive")
@@
 			(layers "*.Cu" "*.Mask")
 			(remove_unused_layers no)
-			(net 1 "/PAIR2")
+			(net 1 "/SW1")
 			(pinfunction "Pin_2")
 			(pintype "passive")
@@
 			(layers "*.Cu" "*.Mask")
 			(remove_unused_layers no)
-			(net 2 "/PAIR3")
+			(net 2 "/SW2")
 			(pinfunction "Pin_3")
 			(pintype "passive")
@@
 			(layers "*.Cu" "*.Mask")
 			(remove_unused_layers no)
-			(net 4 "/PAIR4")
+			(net 4 "/SW3")
 			(pinfunction "Pin_4")
 			(pintype "passive")
@@
 			(remove_unused_layers no)
 			(roundrect_rratio 0.25)
-			(net 3 "/PAIR1")
+			(net 3 "/+24V")
 			(pintype "passive")
 		)
@@
 			(layers "*.Cu" "*.Mask")
 			(remove_unused_layers no)
-			(net 3 "/PAIR1")
+			(net 3 "/+24V")
 			(pintype "passive")
 		)
@@
 			(layers "*.Cu" "*.Mask")
 			(remove_unused_layers no)
-			(net 1 "/PAIR2")
+			(net 1 "/SW1")
 			(pintype "passive")
 		)
@@
 			(layers "*.Cu" "*.Mask")
 			(remove_unused_layers no)
-			(net 2 "/PAIR3")
+			(net 2 "/SW2")
 			(pintype "passive")
 		)
@@
 			(layers "*.Cu" "*.Mask")
 			(remove_unused_layers no)
-			(net 2 "/PAIR3")
+			(net 2 "/SW2")
 			(pintype "passive")
 		)
@@
 			(layers "*.Cu" "*.Mask")
 			(remove_unused_layers no)
-			(net 1 "/PAIR2")
+			(net 1 "/SW1")
 			(pintype "passive")
 		)
@@
 			(layers "*.Cu" "*.Mask")
 			(remove_unused_layers no)
-			(net 4 "/PAIR4")
+			(net 4 "/SW3")
 			(pintype "passive")
 		)
@@
 			(layers "*.Cu" "*.Mask")
 			(remove_unused_layers no)
-			(net 4 "/PAIR4")
+			(net 4 "/SW3")
 			(pintype "passive")
 		)
