File: V2/eumesmo-brk-1ch-v2.kicad_sch (KiCad schematic)
At the start: 2 parts, among them J1 RJ45, J2 1x4P 5,08 SCREW

Commit message: V2.0.0 created
Parts:
- J2: value 1x4P 5,08 SCREW -> 250-204; footprint Tales:TerminalBlock_Dibo_DB128L-5.08-4P_1x04_P5.08mm_Horizontal -> Tales:TerminalBlock_Wago_250-204_1x04_P3.5mm_45Degree; LCSC Part C2915641 -> C2765063; Mfr DIBO -> Wago; Mfr PN DB128V-5.08-4P-GN-S -> 250-204; Vendor PN C2915641 -> C2765063
Other:
- title: 1 Channel RJ45 Breakout Board -> eumesmo 1 Channel RJ45 Breakout Board
Changed lines of the file:
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@@
 	(paper "A4")
 	(title_block
-		(title "1 Channel RJ45 Breakout Board")
-		(date "2022-04-01")
-		(rev "V1")
+		(title "eumesmo 1 Channel RJ45 Breakout Board")
+		(date "2026-06-14")
+		(rev "V2.0")
 	)
 	(text "OPÇÕES RJ45 HORIZONTAL\n\nAMPHENOL RJHSE5080\nMOUSER 523-RJHSE-5080\n\nCKMTW(Shenzhen Cankemeng) R-RJ45R08P-A004\nJLCPCB C385834\n"
@@
 		)
 		(instances
-			(project "eumesmo-brk-1ch-v1"
+			(project "eumesmo-brk-1ch-v2"
 				(path "/78f88cf6-751c-4e9b-ae75-fb8b6d44ff39"
 					(reference "J1")
@@
 			)
 		)
-		(property "Value" "1x4P 5,08 SCREW"
+		(property "Value" "250-204"
 			(at 172.72 102.235 0)
 			(show_name no)
@@
 			)
 		)
-		(property "Footprint" "Tales:TerminalBlock_Dibo_DB128L-5.08-4P_1x04_P5.08mm_Horizontal"
+		(property "Footprint" "Tales:TerminalBlock_Wago_250-204_1x04_P3.5mm_45Degree"
 			(at 170.18 99.06 0)
 			(hide yes)
@@
 			)
 		)
-		(property "LCSC Part" "C2915641"
-			(at 170.18 99.06 0)
-			(hide yes)
-			(show_name no)
-			(do_not_autoplace no)
-			(effects
-				(font
-					(size 1.27 1.27)
-				)
-			)
-		)
-		(property "Mfr" "DIBO"
-			(at 170.18 99.06 0)
-			(hide yes)
-			(show_name no)
-			(do_not_autoplace no)
-			(effects
-				(font
-					(size 1.27 1.27)
-				)
-			)
-		)
-		(property "Mfr PN" "DB128V-5.08-4P-GN-S"
+		(property "LCSC Part" "C2765063"
+			(at 170.18 99.06 0)
+			(hide yes)
+			(show_name no)
+			(do_not_autoplace no)
+			(effects
+				(font
+					(size 1.27 1.27)
+				)
+			)
+		)
+		(property "Mfr" "Wago"
+			(at 170.18 99.06 0)
+			(hide yes)
+			(show_name no)
+			(do_not_autoplace no)
+			(effects
+				(font
+					(size 1.27 1.27)
+				)
+			)
+		)
+		(property "Mfr PN" "250-204"
 			(at 170.18 99.06 0)
 			(hide yes)
@@
 			)
 		)
-		(property "Vendor PN" "C2915641"
+		(property "Vendor PN" "C2765063"
 			(at 170.18 99.06 0)
 			(hide yes)
@@
 		)
 		(instances
-			(project "eumesmo-brk-1ch-v1"
+			(project "eumesmo-brk-1ch-v2"
 				(path "/78f88cf6-751c-4e9b-ae75-fb8b6d44ff39"
 					(reference "J2")
